File: rigol-psu-usb-type-c-adapter.kicad_pcb (KiCad board)
At the start: 2 copper layers, 49 x 27 mm, 12 parts, among them J1 USB_C_Receptacle_USB2.0, J2 Rigol, J3 USB_C_Receptacle_USB2.0

Commit message: Fix CC pull-ups
Memory fooled me. They need to be 10kR, not 5.1kR.
Parts:
- R2, R3, R4, R5: value 5.1kR -> 10kR
Changed lines of the file:
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@@
       (effects (font (size 1 1) (thickness 0.15)))
     )
-    (fp_text value 5.1kR (at 0 1.17) (layer F.Fab)
+    (fp_text value 10kR (at 0 1.17) (layer F.Fab)
       (effects (font (size 1 1) (thickness 0.15)))
     )
@@
       (effects (font (size 1 1) (thickness 0.15)))
     )
-    (fp_text value 5.1kR (at 0 1.17) (layer F.Fab)
+    (fp_text value 10kR (at 0 1.17) (layer F.Fab)
       (effects (font (size 1 1) (thickness 0.15)))
     )
@@
       (effects (font (size 1 1) (thickness 0.15)))
     )
-    (fp_text value 5.1kR (at 0 1.17) (layer F.Fab)
+    (fp_text value 10kR (at 0 1.17) (layer F.Fab)
       (effects (font (size 1 1) (thickness 0.15)))
     )
@@
       (effects (font (size 1 1) (thickness 0.15)))
     )
-    (fp_text value 5.1kR (at 0 1.17) (layer F.Fab)
+    (fp_text value 10kR (at 0 1.17) (layer F.Fab)
       (effects (font (size 1 1) (thickness 0.15)))
     )
